File: Data Pro/data_proV2.brd (EAGLE design)
At the start: 100 x 78.7 mm, 43 parts, among them IC1 4049N, IC2 MCP3008, IC3 OP11S, IC4 LM340MP-05, IC6 AT24CP, J1 RASPBERRYPI-40-PIN-GPIO, U1 DS18B20, X1 32.768khz

Commit message: Data pro update and Lewis' python code
Parts:
- removed IC4: LM340MP-05, linear:SOT223
- added J10: (no value), SparkFun-Connectors:1X02
- B1: value (none) -> CR2032
Connections:
- removed net GPIO0: JP2.6
- removed net GPIO2: JP2.4
- removed net IRQ: JP1.8
- removed net N$13: IC1.2
- removed net N$21: IC1.4
- removed net N$22: IC1.6
- removed net N$23: IC1.10
- removed net RST: JP2.5
- removed net S1-10V: J2.6, J3.6, J4.6, J5.6
- removed net VCC: IC6.8
- new net D1: IC1.2, J1.29
- new net D2: IC1.4, J1.31
- new net D3: IC1.6, J1.32
- new net D4: IC1.10, J1.33
- net 3.3V: now also IC6.8, JP2.5
- net 5V: now also J10.1; no longer IC4.3
- net GND: now also J10.2; no longer IC4.4
Routing:
- net S1-10V: track 62.9 -> 0.00 mm
- net D4: track 0.00 -> 23.7 mm
- net GND: track 539.5 -> 554.9 mm
- net 3.3V: track 227.8 -> 224.0 mm
- net 5V: track 353.0 -> 354.6 mm
