File: Data Pro/data_proV2.sch (EAGLE design)
At the start: 31 parts, among them IC1 4049N, IC2 MCP3008, IC3 OP11S, IC4 LM340MP-05, J1 RASPBERRYPI-40-PIN-GPIO, U1 DS18B20

Commit message: Data pro schematic 11/28/16
Parts:
- removed BAT1, BAT2, BAT3, BAT4: (no value), SparkFun-Electromechanical:BATTERYAA
- added B1: (no value), adafruit:CR2032SMT
- added C1, C2: 0.1uFd, resistor:C-USC0805
- added D3: (no value), SparkFun-DiscreteSemi:DIODESMB
- added IC6: AT24CP, atmel:AT24CP
- added JP2: (no value), adafruit:PINHD-2X4
- added LED1: (no value), led:LEDCHIP-LED0805
- added R10: N/A?, adafruit:R-US_R0805
- added R11, R15, R16: 3.3k, adafruit:R-US_R0805
- added R12: 200, adafruit:R-US_R0805
- added R13: 1.5M, adafruit:R-US_R0805
- added R14: 510K, adafruit:R-US_R0805
- added R17: 1k, adafruit:R-US_R0805
- added X1: 32.768khz, crystal:CRYSTALTC38H
Connections:
- net RIRQ renamed IRQ
- removed net N$9: BAT1.-, BAT2.-, BAT3.-, BAT4.-, IC4.VI
- removed net RCE: JP1.3
- removed net RCSN: JP1.4
- removed net RMISO: JP1.7
- removed net RMOSI: JP1.6
- removed net RSCK: JP1.5
- new net BATT: R13.2, R14.1, U$2.VBATT
- new net CE: J1.GP25, JP1.3
- new net CSN: IC2./CS, J1.CE0, JP1.4
- new net GPIO0: JP2.6
- new net GPIO2: JP2.4
- new net MISO: IC2.DOUT, J1.MISO, JP1.7
- new net MOSI: IC2.DIN, J1.MOSI, JP1.6
- new net N$10: D3.A, R12.1
- new net N$17: LED1.C, R17.2
- new net RST: JP2.5
- new net RX: J1.RXI, JP2.8
- new net SCK: IC2.CLK, J1.SCLK, JP1.5
- new net SCL: IC6.SCL, R16.2, U$2.SCL
- new net SDA: IC6.SDA, R15.2, U$2.SDA
- new net SQ: R11.1, U$2.SQW
- new net TX: J1.TXO, JP2.1
- net 3.3V: now also JP2.3, JP2.7
- net 5V: now also C1.1, C2.1, R10.2, R11.2, R12.2, R15.1, R16.1, U$2.VCC
- net DQ: now also J1.GP27, R9.1
- net GND: now also B1.-, C1.2, C2.2, IC6.A0, IC6.A1, IC6.A2, IC6.GND, IC6.WP, JP2.2, R13.1, R17.1, U$2.GND; no longer BAT1.+, BAT2.+, BAT3.+, BAT4.+
- net N$1: now also U$2.X2, X1.1; no longer IC2.CLK, J1.SCLK
- net N$2: now also R10.1, U$2.X1, X1.2; no longer IC2.DOUT, J1.MISO
- net N$3: now also B1.+, B1.+1, D3.C, R14.2; no longer IC2.DIN, J1.MOSI
- net N$4: now also J1.GP4, LED1.A; no longer IC2./CS, J1.CE0
Other:
- moved on the sheet: U$1

Commit message: Data pro update and Lewis' python code
Parts:
- removed IC4: LM340MP-05, linear:LM340MP-05
- added J10: (no value), SparkFun-Connectors:M02PTH
- B1: value (none) -> CR2032
Connections:
- removed net GPIO0: JP2.6
- removed net GPIO2: JP2.4
- removed net IRQ: JP1.8
- removed net N$13: IC1A.O
- removed net N$21: IC1B.O
- removed net N$22: IC1C.O
- removed net N$23: IC1D.O
- removed net RST: JP2.5
- removed net S1-10V: J2.6, J3.6, J4.6, J5.6
- new net D1: IC1A.O, J1.GP5
- new net D2: IC1B.O, J1.GP6
- new net D3: IC1C.O, J1.GP12
- new net D4: IC1D.O, J1.GP13
- net 3.3V: now also IC6.VCC, JP2.5
- net 5V: now also J10.1; no longer IC4.VO
- net GND: now also J10.2; no longer IC4.GND
Other:
- moved on the sheet: JP2
