File: Data Pro/data_proV3.sch (EAGLE design)
At the start: 45 parts, among them IC1 4049N, IC2 MCP3008, IC3 OP11S, IC4 LM340MP-05, IC6 AT24CP, J1 RASPBERRYPI-40-PIN-GPIO, U1 DS18B20, U2 ESP8266

Commit message: Data pro update and Lewis' python code
Parts:
- removed BAT1, BAT2, BAT3, BAT4: (no value), SparkFun-Electromechanical:BATTERYAA
- removed IC4: LM340MP-05, linear:LM340MP-05
- added C3: 22uF, CH_passive:CAP0805
- added C4, C5: 0.1uF, SparkFun:CAP0603-CAP
- added C6: 10uF, CH_passive:CAP1206
- added JP2: (no value), adafruit:PINHD-2X4
- added JP3: JST, SparkFun:M02-JST-2MM-SMT
- added JP4: VOUT, SparkFun:M02PTH
- added JP7: VIN, SparkFun:M02PTH
- added L1: 4.7uH, 1.2A, SparkFun:INDUCTOR.
- added LED1: (no value), led:LEDCHIP-LED0805
- added R17: 1k, adafruit:R-US_R0805
- added R18, R22: 2M, SparkFun:RESISTOR0603-RES
- added R19, R21: 220k, SparkFun:RESISTOR0603-RES
- added R20: 1.2M, SparkFun:RESISTOR0603-RES
- added SJ1: (no value), SparkFun:SOLDERJUMPER_2WAYPASTE2&3
- B1: value (none) -> CR2032
- R10: value (none) -> N/A?
- R11, R15, R16: value (none) -> 3.3k
- R12: value (none) -> 200
- R13: value (none) -> 1.5M
- R14: value (none) -> 510K
- U2: value ESP8266 -> TPS61200; device SparkFun-RF:ESP8266 -> SparkFun:TPS61200
- X1: value (none) -> 32.768khz
Connections:
- removed net IRQ: JP1.8
- removed net N$21: IC1B.O
- removed net N$22: IC1C.O
- removed net N$23: IC1D.O
- removed net S1-10V: J2.6, J3.6, J4.6, J5.6
- new net D1: IC1A.O, J1.GP5
- new net D2: IC1B.O, J1.GP6
- new net D3: IC1C.O, J1.GP12
- new net D4: IC1D.O, J1.GP13
- new net FB: R21.2, SJ1.2, U2.FB
- new net N$17: LED1.C, R17.2
- new net N$4: J1.GP4, LED1.A
- new net RX: J1.RXI, JP2.8
- new net TX: J1.TXO, JP2.1
- new net UVLO: C4.2, R18.1, R19.2, U2.UVLO
- new net VCC: C3.1, JP4.2, R20.2, R22.2, U2.VOUT
- new net VIN: C4.1, C6.1, JP3.2, JP7.2, L1.2, R18.2, U2.EN, U2.PS, U2.VIN
- net 3.3V: now also IC6.VCC, JP2.3, JP2.5, JP2.7, R20.1, SJ1.1
- net 5V: now also R22.1, SJ1.3; no longer IC4.VO
- net DQ: now also J1.GP27, R9.1
- net GND: now also C3.2, C5.2, C6.2, JP2.2, JP3.1, JP4.1, JP7.1, R17.1, R19.1, R21.1, U2.GND, U2.PAD@1, U2.PAD@2, U2.PAD@3, U2.PAD@4, U2.PAD@5, U2.PGND; no longer BAT1.+, BAT2.+, BAT3.+, BAT4.+, IC4.GND
- net N$13: now also C5.1, U2.VAUX; no longer IC1A.O
- net N$9: now also L1.1, U2.L; no longer BAT1.-, BAT2.-, BAT3.-, BAT4.-, IC4.VI
Other:
- note added: "UVLO 2.6V"
- moved on the sheet: B1, C1, C2, D3, IC6, JP1, R10, R11, R12, R13, R14, R15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
