File: Data Pro/data_proV1.1.sch (EAGLE design)
At the start: 57 parts, among them IC1 4049N, IC2 MCP3008, IC3 OP11S, IC6 AT24CP, J1 RASPBERRYPI-40-PIN-GPIO, U1 DS18B20, U2 TPS61200, X1 32.768khz

Commit message: Data pro update v1.2
The schematic is complete, working on the board.
Parts:
- removed JP3: JST, SparkFun:M02-JST-2MM-SMT
- removed JP7: VIN, SparkFun:M02PTH
- added BATT: (no value), adafruit:JST_2PIN-SMT-RA
- added C10: 4700uF/10V, adafruit:CPOL-USE5-13
- added C7, C8, C9: 10uF, adafruit:C-USC0805K
- added CHRG/LBO: ORANGE, microbuilder:LED0805_NOOUTLINE
- added CN1: DCIN, microbuilder:DCBARRELSMT
- added CN4: USB-MINIB-5PIN, SparkFun-Connectors:USB-MINIB-5PIN
- added D2: MBR120VLSFT1G, microbuilder:DIODESOD-123
- added DONE: GREEN, microbuilder:LED0805_NOOUTLINE
- added IC4: MCP73871, adafruit:MCP73871
- added JP6: BATT, microbuilder:HEADER-1X2ROUND
- added LOAD: JST-O, adafruit:JST_2PIN-SMT-RA
- added PWR: RED, microbuilder:LED0805_NOOUTLINE
- added R23: 270K, adafruit:R-US_R0805
- added R24, R29: 100K, adafruit:R-US_R0805
- added R25, R26, R27: 1K, adafruit:R-US_R0805
- added R28: 2K, adafruit:R-US_FLIPFLOP
- added R30: 1K, adafruit:R-US_M0805
- added R31: 0, adafruit:R-US_R0805
- added RT2: 150K, adafruit:R-US_M0805
- added THERM: 10K, adafruit:R-US_FLIPFLOP
- D1, D3, LED1: value (none) -> 0805 CHIP
- J2, J3, J4, J5: value (none) -> BTA
- J6, J7, J8, J9: value (none) -> BTD
- JP1: value (none) -> NRF24L01
- JP2: value (none) -> ESP8266
- JP4: value VOUT -> DCIN; device SparkFun:M02PTH -> microbuilder:HEADER-1X2
- R1, R2, R3, R4, R5, R6, R7, R8: value (none) -> 1k
- R10: value N/A? -> 1k
Connections:
- removed net 3.3V: D1.C, IC6.VCC, J1.3.3V@1, J1.3.3V@17, JP1.2, JP2.3, JP2.5, JP2.7, R20.1, SJ1.1, U$1.OUT, U1.VDD
- removed net 5V: C1.1, C2.1, IC2.VDD, IC2.VREF, J1.5V@2, J1.5V@4, J2.5, J3.5, J4.5, J5.5, J6.4, J7.4, J8.4, J9.4, R10.2, R11.2, R12.2, R15.1, R16.1, R22.1, SJ1.3, U$1.IN, U$2.VCC
- removed net VCC: C3.1, JP4.2, R20.2, R22.2, U2.VOUT
- new net BATT1: BATT.2, C8.1, IC4.VBAT1, IC4.VBAT2, IC4.VBAT3, JP6.1
- new net N$18: IC4.VPCC, R23.1, R24.1
- new net N$19: IC4./PG, PWR.C
- new net N$20: DONE.C, IC4.STAT2
- new net N$21: CHRG/LBO.C, IC4.STAT1/LBO
- new net N$22: CHRG/LBO.A, R25.1
- new net N$23: DONE.A, R26.1
- new net N$24: PWR.A, R27.1
- new net N$25: IC4.PROG3, R29.2
- new net N$26: IC4.PROG1, R28.2
- new net N$27: IC4.THERM, R30.1
- new net N$28: R30.2, RT2.2, THERM.2
- new net N$29: CN1.PWR, D2.A
- new net N$30: CN4.VBUS, R31.1
- new net N$31: CN1.GND, CN4.GND
- new net VDD: D1.C, J1.3.3V@1, J1.3.3V@17, JP1.2, JP2.3, JP2.5, JP2.7, R20.1, SJ1.1, U$1.OUT, U1.VDD
- new net VOUT: C1.1, C10.+, C2.1, C3.1, C9.1, D2.C, IC2.VDD, IC2.VREF, IC4./TE, IC4.CE, IC4.IN1, IC4.IN2, IC4.PROG2, IC4.SEL, IC6.VCC, J1.5V@2, J1.5V@4, J2.5, J3.5, J4.5, J5.5, J6.4, J7.4, J8.4, J9.4, JP4.2, R10.2, R11.2, R12.2, R15.1, R16.1, R20.2, R22.1, R22.2, R23.2, R25.2, R26.2, R27.2, R31.2, SJ1.3, U$1.IN, U$2.VCC, U2.VOUT
- net GND: now also BATT.1, C10.-, C7.2, C8.2, C9.2, CN1.GNDBREAK, IC4.GND1, IC4.GND2, IC4.GND3, JP6.2, LOAD.1, R24.2, R28.1, R29.1, RT2.1, THERM.1; no longer JP3.1, JP7.1
- net VIN: now also C7.1, IC4.OUT1, IC4.OUT2, LOAD.2; no longer JP3.2, JP7.2
Other:
- note added: "1.0K = 1000mA"
- note added: "10K NTC Thermistor:"
- note added: "2.0K = 500mA"
- note added: "Charge Rate = 1000V/PROG1"
- note added: "No Thermistor:"
- note added: "RT1 = 0, RT2 = 10K"
- note added: "RT1 = TBD, RT2 = TBD"
- moved on the sheet: JP4, LED1, U$1
