File: Data Pro/data_proV1.2.brd (EAGLE design)
At the start: 100 x 80 mm, 75 parts, among them CN1 DCIN, IC1 4049N, IC2 MCP3008, IC3 LM324D, IC4 MCP73871, IC6 AT24CP, J1 RASPBERRYPI-40-PIN-GPIO, J2 A2, J3 A3, J4 A4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

Commit message: Data pro update v1.2 (Complete)
Parts:
- moved R18 19.1 mm to (45.7, 26.7), turned to 270 degrees
- moved C4 16.1 mm to (42.5, 26.7), turned to 90 degrees
- moved R19 14.4 mm to (38.7, 27.3), turned to 0 degrees
- moved C3 14.3 mm to (31.8, 21.0), turned to 270 degrees
- moved R22 13.6 mm to (28.6, 26.7), turned to 180 degrees
- moved R20 9.03 mm to (26.0, 23.5), turned to 270 degrees
- moved DONE 8.89 mm to (61.6, 8.89)
- moved R26 8.89 mm to (61.6, 3.81)
- moved C6 7.96 mm to (40.0, 21.6), turned to 270 degrees
- moved C5 7.75 mm to (28.6, 21.0), turned to 0 degrees
- moved R8 7.62 mm to (57.1, 41.9)
- moved L1 7.10 mm to (36.8, 17.1), turned to 0 degrees
- moved SJ1 6.84 mm to (31.8, 25.4), turned to 90 degrees
- moved IC3 6.48 mm to (49.5, 47.0)
- moved R1 6.48 mm to (38.1, 49.5)
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Routing:
- net 3.3V: track 188.2 -> 129.0 mm
- net MOSI: track 31.1 -> 78.4 mm, vias 0 -> 1
- net D4: track 80.5 -> 116.6 mm
- net DQ: track 68.0 -> 36.7 mm, vias 5 -> 0
- net SCK: track 37.4 -> 68.5 mm, vias 0 -> 3
- net VCC: track 83.4 -> 114.0 mm, vias 3 -> 2
- net CSN: track 72.6 -> 96.7 mm
- net GND: track 631.5 -> 610.2 mm, vias 2 -> 1
- net D3: track 67.7 -> 89.0 mm, vias 0 -> 1
- net N$18: track 0.00 -> 18.9 mm
- net MISO: track 87.8 -> 69.9 mm, vias 3 -> 1
- net S1-5V2: track 67.2 -> 49.8 mm, vias 3 -> 1
- net N$3: track 62.6 -> 46.1 mm, vias 2 -> 1
- net N$13: track 0.00 -> 15.7 mm, vias 0 -> 2
- net 5V: track 408.5 -> 393.5 mm, vias 3 -> 4
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
Commit message: Data pro complete
Parts:
- removed JP1: NRF24L01, pinhead:2X04
- added M1: WIRELESS-NRF24L01, diy-modules:WIRELESS-NRF24L01
- moved JP2 58.5 mm to (85.1, 5.08), turned to 180 degrees
Connections:
- net 3.3V: now also M1.2; no longer JP1.2
- net CE: now also M1.3; no longer JP1.3
- net CSN: now also M1.4; no longer JP1.4
- net GND: now also M1.1; no longer JP1.1
- net MISO: now also M1.7; no longer JP1.7
- net MOSI: now also M1.6; no longer JP1.6
- net SCK: now also M1.5; no longer JP1.5
Routing:
- net TX: track 20.4 -> 248.7 mm, vias 0 -> 1
- net RX: track 11.7 -> 81.6 mm, vias 0 -> 1
- net 3.3V: track 129.0 -> 193.9 mm, vias 2 -> 3
- net GND: track 610.2 -> 639.8 mm, vias 1 -> 0
- net CE: track 41.1 -> 20.3 mm
- net MISO: track 69.9 -> 90.4 mm, vias 1 -> 2
- net CSN: track 96.7 -> 116.1 mm, vias 0 -> 1
- net D1: track 64.2 -> 83.4 mm, vias 1 -> 3
- net D3: track 89.0 -> 75.4 mm, vias 1 -> 3
- net SCK: track 68.5 -> 62.5 mm
- net DQ: track 36.7 -> 33.9 mm, vias 0 -> 2
- net MOSI: track 78.4 -> 75.9 mm, vias 1 -> 4

Commit message: More data pro updates
Sorry
Parts:
- moved PWR 2.62 mm to (55.2, 8.26), turned to 90 degrees
Connections:
- net CE: now also J1.15; no longer J1.22
Routing:
- net CE: track 20.3 -> 11.4 mm
- net VCC: track 114.0 -> 111.9 mm
- net N$24: track 3.03 -> 4.06 mm
- net N$20: track 8.58 -> 9.39 mm
- net BATT1: track 25.0 -> 25.5 mm
- net N$25: track 7.99 -> 8.52 mm
- net VIN: track 54.0 -> 54.5 mm
- net N$19: track 5.55 -> 5.04 mm
Changed lines of the file:
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@@
 </element>
 <element name="LED1" library="led" package="CHIP-LED0805" value="" x="82.55" y="76.2" rot="R270"/>
-<element name="PWR" library="microbuilder" package="CHIPLED_0805_NOOUTLINE" value="RED" x="57.785" y="8.89" smashed="yes">
-<attribute name="NAME" x="56.769" y="7.112" size="0.8128" layer="25" ratio="18" rot="R90"/>
+<element name="PWR" library="microbuilder" package="CHIPLED_0805_NOOUTLINE" value="RED" x="55.245" y="8.255" smashed="yes" rot="R90">
+<attribute name="NAME" x="57.023" y="7.239" size="0.8128" layer="25" ratio="18" rot="R180"/>
 </element>
 <element name="R1" library="resistor" package="R0805" value="1k" x="38.1" y="49.53" smashed="yes">
@@
 <attribute name="NAME" x="10.795" y="69.342" size="1.27" layer="25" ratio="10" rot="R90"/>
 </element>
-<element name="M1" library="diy-modules" package="WIRELESS-NRF24L01" value="WIRELESS-NRF24L01" x="72.39" y="59.69"/>
+<element name="M1" library="diy-modules" package="WIRELESS-NRF24L01" value="WIRELESS-NRF24L01" x="72.39" y="59.69" smashed="yes">
+<attribute name="NAME" x="72.39" y="68.58" size="1.27" layer="25" align="bottom-center"/>
+</element>
 </elements>
 <signals>
@@
 </signal>
 <signal name="CE">
-<contactref element="J1" pad="22"/>
 <contactref element="M1" pad="3"/>
 <wire x1="48.26" y1="63.5" x2="59.69" y2="63.5" width="0.254" layer="16"/>
-<wire x1="48.26" y1="72.39" x2="48.26" y2="63.5" width="0.254" layer="1"/>
 <via x="48.26" y="63.5" extent="1-16" drill="0.6096"/>
+<contactref element="J1" pad="15"/>
+<wire x1="59.69" y1="63.5" x2="55.88" y2="74.93" width="0" layer="19" extent="1-1"/>
 </signal>
 <signal name="N$6">
@@
 <wire x1="42.965" y1="25.4" x2="43.18" y2="25.4" width="0.254" layer="1"/>
 <wire x1="35.56" y1="23.065" x2="35.56" y2="24.13" width="0.254" layer="1"/>
-<wire x1="35.56" y1="24.13" x2="36.83" y2="25.4" width="0.254" layer="1"/>
-<wire x1="36.83" y1="25.4" x2="39.37" y2="25.4" width="0.254" layer="1"/>
 <wire x1="39.37" y1="25.4" x2="40.005" y2="24.765" width="0.254" layer="1"/>
 <wire x1="40.005" y1="24.765" x2="40.005" y2="22.99" width="0.254" layer="1"/>
@@
 <via x="43.18" y="20.32" extent="1-16" drill="0.6"/>
 <wire x1="40.64" y1="22.86" x2="43.18" y2="20.32" width="0.254" layer="1"/>
+<wire x1="35.56" y1="24.13" x2="37.465" y2="26.035" width="0.254" layer="1"/>
+<wire x1="37.465" y1="26.035" x2="38.735" y2="26.035" width="0.254" layer="1"/>
+<wire x1="38.735" y1="26.035" x2="39.37" y2="25.4" width="0.254" layer="1"/>
 </signal>
 <signal name="N$17">
@@
 <via x="52.86375" y="17.93875" extent="1-16" drill="0.6096"/>
 <wire x1="57.785" y1="2.81" x2="61.595" y2="2.81" width="0.4064" layer="1"/>
-<wire x1="55.745" y1="13.275" x2="55.88" y2="13.14" width="0.254" layer="1"/>
-<wire x1="55.88" y1="13.14" x2="55.88" y2="12.7" width="0.254" layer="1"/>
-<wire x1="55.88" y1="12.7" x2="56.515" y2="12.7" width="0.254" layer="1"/>
-<wire x1="56.515" y1="12.7" x2="57.15" y2="12.065" width="0.254" layer="1"/>
-<wire x1="57.15" y1="12.065" x2="59.055" y2="12.065" width="0.254" layer="1"/>
-<via x="59.055" y="12.065" extent="1-16" drill="0.6"/>
-<wire x1="59.055" y1="12.065" x2="57.15" y2="10.16" width="0.254" layer="16"/>
-<wire x1="57.15" y1="10.16" x2="46.99" y2="10.16" width="0.254" layer="16"/>
 <wire x1="46.99" y1="10.16" x2="46.0375" y2="11.1125" width="0.254" layer="16"/>
+<wire x1="55.745" y1="13.275" x2="55.745" y2="12.2" width="0.254" layer="1"/>
+<wire x1="55.745" y1="12.2" x2="55.88" y2="12.065" width="0.254" layer="1"/>
+<wire x1="55.88" y1="12.065" x2="56.515" y2="12.065" width="0.254" layer="1"/>
+<wire x1="56.515" y1="12.065" x2="57.15" y2="12.7" width="0.254" layer="1"/>
+<via x="57.15" y="12.7" extent="1-16" drill="0.6"/>
+<wire x1="57.15" y1="12.7" x2="57.15" y2="11.43" width="0.254" layer="16"/>
+<wire x1="57.15" y1="11.43" x2="55.88" y2="10.16" width="0.254" layer="16"/>
+<wire x1="55.88" y1="10.16" x2="46.99" y2="10.16" width="0.254" layer="16"/>
 </signal>
 <signal name="N$18">
@@
 <contactref element="PWR" pad="C"/>
 <contactref element="IC4" pad="P$6"/>
-<wire x1="54.13375" y1="12.54125" x2="54.13375" y2="13.17625" width="0.254" layer="1"/>
-<wire x1="56.67375" y1="10.00125" x2="54.13375" y2="12.54125" width="0.254" layer="1"/>
-<wire x1="57.785" y1="10.00125" x2="56.67375" y2="10.00125" width="0.254" layer="1"/>
-<wire x1="54.13375" y1="13.17625" x2="54.245" y2="13.275" width="0.254" layer="1"/>
-<wire x1="57.785" y1="10.00125" x2="57.785" y2="9.94" width="0.254" layer="1"/>
+<wire x1="54.195" y1="8.255" x2="54.195" y2="13.225" width="0.254" layer="1"/>
+<wire x1="54.195" y1="13.225" x2="54.245" y2="13.275" width="0.254" layer="1"/>
 </signal>
 <signal name="N$20">
 <contactref element="IC4" pad="P$7"/>
 <contactref element="DONE" pad="C"/>
-<wire x1="54.76875" y1="12.7" x2="54.76875" y2="13.17625" width="0.254" layer="1"/>
-<wire x1="56.515" y1="10.95375" x2="54.76875" y2="12.7" width="0.254" layer="1"/>
-<wire x1="60.6425" y1="10.95375" x2="56.515" y2="10.95375" width="0.254" layer="1"/>
-<wire x1="61.595" y1="10.00125" x2="60.6425" y2="10.95375" width="0.254" layer="1"/>
-<wire x1="54.76875" y1="13.17625" x2="54.745" y2="13.275" width="0.254" layer="1"/>
-<wire x1="61.595" y1="10.00125" x2="61.595" y2="9.94" width="0.254" layer="1"/>
+<wire x1="61.595" y1="9.94" x2="60.74" y2="10.795" width="0.254" layer="1"/>
+<wire x1="60.74" y1="10.795" x2="55.245" y2="10.795" width="0.254" layer="1"/>
+<wire x1="55.245" y1="10.795" x2="54.745" y2="11.295" width="0.254" layer="1"/>
+<wire x1="54.745" y1="11.295" x2="54.745" y2="13.275" width="0.254" layer="1"/>
 </signal>
 <signal name="N$21">
@@
 <contactref element="CHRG/LBO" pad="C"/>
 <wire x1="65.405" y1="9.94" x2="63.915" y2="11.43" width="0.254" layer="1"/>
-<wire x1="63.915" y1="11.43" x2="57.15" y2="11.43" width="0.254" layer="1"/>
-<wire x1="57.15" y1="11.43" x2="56.515" y2="12.065" width="0.254" layer="1"/>
-<wire x1="56.515" y1="12.065" x2="55.88" y2="12.065" width="0.254" layer="1"/>
-<wire x1="55.88" y1="12.065" x2="55.245" y2="12.7" width="0.254" layer="1"/>
-<wire x1="55.245" y1="12.7" x2="55.245" y2="13.275" width="0.254" layer="1"/>
+<wire x1="55.245" y1="13.275" x2="55.245" y2="12.065" width="0.254" layer="1"/>
+<wire x1="55.245" y1="12.065" x2="55.88" y2="11.43" width="0.254" layer="1"/>
+<wire x1="55.88" y1="11.43" x2="63.915" y2="11.43" width="0.254" layer="1"/>
 </signal>
 <signal name="N$22">
@@
 <contactref element="PWR" pad="A"/>
 <contactref element="R27" pad="1"/>
-<wire x1="57.785" y1="4.81" x2="57.785" y2="7.84" width="0.254" layer="1"/>
+<wire x1="57.785" y1="4.81" x2="57.785" y2="6.765" width="0.254" layer="1"/>
+<wire x1="57.785" y1="6.765" x2="56.295" y2="8.255" width="0.254" layer="1"/>
 </signal>
 <signal name="N$25">
 <contactref element="IC4" pad="P$12"/>
 <contactref element="R29" pad="2"/>
-<wire x1="60.16625" y1="14.76375" x2="57.30875" y2="14.76375" width="0.254" layer="1"/>
-<wire x1="63.65875" y1="14.76375" x2="60.16625" y2="14.76375" width="0.254" layer="16"/>
 <wire x1="62.38875" y1="14.76375" x2="63.65875" y2="14.76375" width="0.254" layer="1"/>
 <wire x1="62.23" y1="14.9225" x2="62.38875" y2="14.76375" width="0.254" layer="1"/>
 <wire x1="57.30875" y1="14.76375" x2="57.21" y2="14.74" width="0.254" layer="1"/>
 <wire x1="62.23" y1="14.9225" x2="62.23" y2="14.97" width="0.254" layer="1"/>
-<via x="60.16625" y="14.76375" extent="1-16" drill="0.6096"/>
+<via x="58.89625" y="14.12875" extent="1-16" drill="0.6096"/>
 <via x="63.65875" y="14.76375" extent="1-16" drill="0.6096"/>
+<wire x1="57.30875" y1="14.76375" x2="58.26125" y2="14.76375" width="0.254" layer="1"/>
+<wire x1="58.26125" y1="14.76375" x2="58.89625" y2="14.12875" width="0.254" layer="1"/>
+<wire x1="58.89625" y1="14.12875" x2="63.02375" y2="14.12875" width="0.254" layer="16"/>
+<wire x1="63.02375" y1="14.12875" x2="63.65875" y2="14.76375" width="0.254" layer="16"/>
 </signal>
 <signal name="N$26">
@@
 <wire x1="72.7075" y1="12.7" x2="72.66" y2="12.7" width="0.254" layer="1"/>
 <wire x1="72.7075" y1="7.62" x2="72.66" y2="8.78" width="0.254" layer="1"/>
-<wire x1="59.055" y1="15.71625" x2="57.30875" y2="15.71625" width="0.254" layer="1"/>
-<wire x1="69.5325" y1="15.71625" x2="59.055" y2="15.71625" width="0.254" layer="16"/>
 <wire x1="72.54875" y1="12.7" x2="69.5325" y2="15.71625" width="0.254" layer="1"/>
 <wire x1="57.30875" y1="15.71625" x2="57.21" y2="15.74" width="0.254" layer="1"/>
 <wire x1="72.54875" y1="12.7" x2="72.66" y2="12.7" width="0.254" layer="1"/>
-<via x="59.055" y="15.71625" extent="1-16" drill="0.6096"/>
+<via x="59.055" y="16.35125" extent="1-16" drill="0.6096"/>
 <via x="69.5325" y="15.71625" extent="1-16" drill="0.6096"/>
+<wire x1="57.30875" y1="15.71625" x2="58.42" y2="15.71625" width="0.254" layer="1"/>
+<wire x1="58.42" y1="15.71625" x2="59.055" y2="16.35125" width="0.254" layer="1"/>
+<wire x1="59.055" y1="16.35125" x2="68.8975" y2="16.35125" width="0.254" layer="16"/>
+<wire x1="68.8975" y1="16.35125" x2="69.5325" y2="15.71625" width="0.254" layer="16"/>
 </signal>
 <signal name="5VO">
